Commit message: Finish rclpy/SimControl env port + consolidated DR + multi-arena render
Completes the ROS 1 Noetic/Gazebo classic -> ROS 2 Lyrical/Gazebo Jetty port
of the env runtime on top of the previously-landed SimControl seam.

Env runtime (rclpy + SimControl, AWS-free):
- rollout_agent_ctrl: ModelState->compat, Float64MultiArray group commands,
  os.environ params, ROS2 clock fields (.sec/.nanosec), DomainRandomizer
  integration (sample/apply in reset, steering_bias + motor_delay in send_action,
  dr_info passthrough).
- deepracer_env / multi_agent_env: build agents via runtime.get_node(); set_world
  through the seam pause/unpause; merge per-arena dr_info into step/reset info.
- sensors_rollout: rclpy subscriptions + optional Gaussian camera/lidar noise.

Consolidated domain randomization (single per-arena source of truth):
- domain_randomizations/spec.py (RandomizationSpec, from_env GYM_DR_*) and
  domain_randomizer.py (sample -> EpisodeRandomization, apply via SimControl):
  start position, CW/CCW direction, visual recolor, lighting, friction,
  steering bias, motor delay, sensor noise. Host tests under tests/.

Live N-car multi-arena (one shared sim, fully decoupled):
- multi_arena.launch.py: N namespaced arenas, each its own controller_manager.
- ros2_control.yaml: /**/-wildcard keys so controllers load under any namespace.
- deepracer_gz.urdf.xacro: include_camera arg (sensorless render cars), per-car
  <ros><namespace> for the gz_ros2_control system plugin.

Real-render tooling (verified GPU OGRE2/EGL):
- docker/Dockerfile.render-gpu (NVIDIA EGL ICD) + Dockerfile.render (llvmpipe).
- examples/_render_capture.py, multi_arena_record.py, render_multiarena_video.py.

Docs: architecture/{domain-randomization,multi-arena}.md, PORTING_STATUS.md.

Co-Authored-By: Claude Opus 4.8 <noreply@anthropic.com>

File: simulation/urdf/deepracer/deepracer_gz.urdf.xacro (robot description, xacro)
@@ -14,4 +14,7 @@
     car_name    : entity / topic namespace (e.g. "car_0") — sensors publish to
                   /<car_name>/camera/... and /<car_name>/scan.
+    namespace   : ROS namespace for this car's gz_ros2_control controller_manager
+                  (default "" = root). Set per-car (e.g. "racecar_1") so N cars
+                  in ONE gz world each get their own /<namespace>/controller_manager.
     friction_mu : wheel friction coefficient (domain-randomisation knob).
     ros2_control_config : absolute path to ros2_control.yaml.
@@ -20,4 +23,6 @@
 <robot name="deepracer" xmlns:xacro="http://www.ros.org/wiki/xacro">
   <xacro:arg name="car_name" default="car"/>
+  <xacro:arg name="namespace" default=""/>
+  <xacro:arg name="include_camera" default="true"/>
   <xacro:arg name="friction_mu" default="1.5"/>
   <xacro:arg name="ros2_control_config"
@@ -25,4 +30,5 @@
   <xacro:arg name="include_lidar" default="true"/>
   <xacro:property name="car_name" value="$(arg car_name)"/>
+  <xacro:property name="namespace" value="$(arg namespace)"/>
   <xacro:property name="mu" value="$(arg friction_mu)"/>
   <xacro:property name="mesh" value="model://meshes/deepracer"/>
@@ -167,19 +173,33 @@
     <plugin filename="gz_ros2_control-system" name="gz_ros2_control::GazeboSimROS2ControlPlugin">
       <parameters>$(arg ros2_control_config)</parameters>
+      <!-- Per-car namespacing: when 'namespace' is non-empty, run this car's
+           controller_manager under that ROS namespace so N cars in ONE gz world
+           don't collide. The fully-qualified node becomes
+           /<namespace>/controller_manager. Do NOT set <controller_manager_name>
+           to "<ns>/controller_manager": gz_ros2_control turns it into a node
+           name remap (-r __node:=...), and a node NAME may not contain '/' — that
+           parse error throws uncaught and aborts the whole gz server. -->
+      <xacro:if value="${namespace != ''}">
+        <ros>
+          <namespace>${namespace}</namespace>
+        </ros>
+      </xacro:if>
     </plugin>
   </gazebo>
-  <gazebo reference="camera_link">
-    <sensor name="zed_camera" type="camera">
-      <topic>${car_name}/camera/zed/rgb/image_rect_color</topic>
-      <gz_frame_id>camera_link</gz_frame_id>
-      <update_rate>15</update_rate>
-      <always_on>1</always_on>
-      <camera>
-        <horizontal_fov>1.13</horizontal_fov>
-        <image><width>640</width><height>480</height><format>R8G8B8</format></image>
-        <clip><near>0.02</near><far>300</far></clip>
-      </camera>
-    </sensor>
-  </gazebo>
+  <xacro:if value="$(arg include_camera)">
+    <gazebo reference="camera_link">
+      <sensor name="zed_camera" type="camera">
+        <topic>${car_name}/camera/zed/rgb/image_rect_color</topic>
+        <gz_frame_id>camera_link</gz_frame_id>
+        <update_rate>15</update_rate>
+        <always_on>1</always_on>
+        <camera>
+          <horizontal_fov>1.13</horizontal_fov>
+          <image><width>640</width><height>480</height><format>R8G8B8</format></image>
+          <clip><near>0.02</near><far>300</far></clip>
+        </camera>
+      </sensor>
+    </gazebo>
+  </xacro:if>
   <xacro:if value="$(arg include_lidar)">
     <gazebo reference="laser">

Commit message: Raise wheel joint velocity limit 100->140 rad/s (max speed needs 114)
The action space allows speed up to 4.0 m/s -> 4.0/0.035 = 114 rad/s wheel
velocity, but the wheel joints capped velocity at 100 rad/s (3.5 m/s). At top
speed gz_ros2_control clamped the command every step ('Command out of limits'),
a discontinuity that can cascade into physics/render instability. Steering
hinges stay at 100 (they don't spin).

Co-Authored-By: Claude Opus 4.8 <noreply@anthropic.com>

File: simulation/urdf/deepracer/deepracer_gz.urdf.xacro (robot description, xacro)
@@ -82,10 +82,10 @@
     <parent link="chassis"/><child link="left_rear_wheel"/>
     <origin xyz="-0.081663 0.08105 0.01575" rpy="0 0 0"/><axis xyz="0 1 0"/>
-    <limit effort="10" velocity="100"/>
+    <limit effort="10" velocity="140"/>
   </joint>
   <joint name="right_rear_wheel_joint" type="continuous">
     <parent link="chassis"/><child link="right_rear_wheel"/>
     <origin xyz="-0.081663 -0.08105 0.01575" rpy="0 0 0"/><axis xyz="0 1 0"/>
-    <limit effort="10" velocity="100"/>
+    <limit effort="10" velocity="140"/>
   </joint>
   <!-- steering hinges: steered (position), about Z, ±1 rad -->
@@ -114,10 +114,10 @@
     <parent link="left_steering_hinge"/><child link="left_front_wheel"/>
     <origin xyz="0 0 0" rpy="0 0 0"/><axis xyz="0 1 0"/>
-    <limit effort="10" velocity="100"/>
+    <limit effort="10" velocity="140"/>
   </joint>
   <joint name="right_front_wheel_joint" type="continuous">
     <parent link="right_steering_hinge"/><child link="right_front_wheel"/>
     <origin xyz="0 0 0" rpy="0 0 0"/><axis xyz="0 1 0"/>
-    <limit effort="10" velocity="100"/>
+    <limit effort="10" velocity="140"/>
   </joint>
   <!-- camera + lidar mount links -->

Commit message: fix(urdf): steering hinges revolute ±30° so the declared limit is real (was continuous → ignored)
The steering hinge joints were type=continuous, so gz_ros_control reported 'no position limits' and the URDF's declared range was meaningless. Made them proper bounded revolute joints at ±0.5236 rad (30°), matching the agent's MAX_STEERING_DEG=30 (deepracer_env/agent_ctrl/drive.py) and the physical car. Found via a real-sim training smoke that spammed gz_ros_control 'left_steering_hinge_joint out of limits'. Validated: the joint now reports 'has position limits: true [-0.5236, 0.5236]' and training runs clean. The residual throttled 'out of limits' warnings during sharp steering reversals are the JointSaturationLimiter's per-tick servo-slew limiting (a held ±30° command settles to the full ±30°), not a static cap.

Co-Authored-By: Claude Opus 4.8 <noreply@anthropic.com>

File: simulation/urdf/deepracer/deepracer_gz.urdf.xacro (robot description, xacro)
@@ -89,5 +89,14 @@
     <limit effort="10" velocity="140"/>
   </joint>
-  <!-- steering hinges: steered (position), about Z, ±1 rad -->
+  <!-- steering hinges: steered (position), about Z. REVOLUTE (bounded) at ±30°
+       (0.5236 rad) — matches the agent's ±30° command (MAX_STEERING_DEG, drive.py)
+       and the real car. Was `type="continuous"`, so gz_ros_control reported "no
+       position limits" and the declared range was meaningless. Revolute makes the
+       ±30° bound real. NOTE: gz_ros_control's JointSaturationLimiter additionally
+       rate-limits sharp steering *reversals* per control tick (logs a throttled
+       "out of limits" while the joint is moving fast the other way) — that's correct
+       servo-slew behaviour, not a static cap: a *held* ±30° command settles to the
+       full ±30° (velocity→0 → limiter allows the bound). Silencing the reversal
+       warnings entirely would need gz_ros_control velocity-limit tuning; benign. -->
   <link name="left_steering_hinge">
     <visual><geometry><mesh filename="${mesh}/left_steering_hinge.STL"/></geometry></visual>
@@ -98,13 +107,13 @@
     <inertial><mass value="0.01"/><inertia ixx="1e-6" iyy="1e-6" izz="1e-6" ixy="0" ixz="0" iyz="0"/></inertial>
   </link>
-  <joint name="left_steering_hinge_joint" type="continuous">
+  <joint name="left_steering_hinge_joint" type="revolute">
     <parent link="chassis"/><child link="left_steering_hinge"/>
     <origin xyz="0.082311 0.079601 0.011759" rpy="0 0 0"/><axis xyz="0 0 1"/>
-    <limit lower="-1" upper="1" effort="10" velocity="100"/>
-  </joint>
-  <joint name="right_steering_hinge_joint" type="continuous">
+    <limit lower="-0.5236" upper="0.5236" effort="10" velocity="100"/>
+  </joint>
+  <joint name="right_steering_hinge_joint" type="revolute">
     <parent link="chassis"/><child link="right_steering_hinge"/>
     <origin xyz="0.082311 -0.079601 0.011759" rpy="0 0 0"/><axis xyz="0 0 1"/>
-    <limit lower="-1" upper="1" effort="10" velocity="100"/>
+    <limit lower="-0.5236" upper="0.5236" effort="10" velocity="100"/>
   </joint>
   <!-- front wheels: children of the steering hinges, roll about Y -->
